Commit message: trying to get rid of warning in colcon build

File: grace_description/urdf/grace.urdf.xacro (robot description, xacro)
@@ -322,4 +322,40 @@
     <axis xyz="0 0 0" />
   </joint>
+  <!-- Camera -->
+  <link name="camera_link">
+    <inertial>
+      <origin xyz="-0.019934 -0.030537 -0.049914" rpy="0 0 0" />
+      <mass value="0.27538" />
+      <inertia ixx="0.00029613" ixy="2.0639E-07" ixz="3.1613E-06"
+               iyy="0.00015935" iyz="9.9814E-09"
+               izz="0.00017529" />
+    </inertial>
+    <visual>
+      <origin xyz="0 0 0" rpy="0 0 0" />
+      <geometry>
+        <mesh filename="package://grace_description/meshes/Camera_Link.STL" />
+      </geometry>
+      <material name="yellow"/>
+    </visual>
+    <collision>
+      <origin xyz="0 0 0" rpy="0 0 0" />
+      <geometry>
+        <mesh filename="package://grace_description/meshes/Camera_Link.STL" />
+      </geometry>
+    </collision>
+  </link>
+  <joint name="camera_joint" type="fixed">
+    <origin xyz="-0.19268 0.030962 0.2792" rpy="0 0 0" />
+    <parent link="base_link" />
+    <child link="camera_link" />
+    <axis xyz="0 0 0" />
+  </joint>
+  <!-- Camera Optical Frame (Z forward, X right, Y down) -->
+  <link name="camera_optical_frame"/>
+  <joint name="camera_optical_joint" type="fixed">
+    <origin xyz="0 0 0" rpy="-1.5708 0 -1.5708" />
+    <parent link="camera_link" />
+    <child link="camera_optical_frame" />
+  </joint>
   <material name="blue">
     <color rgba="0 0 1 1"/>
@@ -334,3 +370,6 @@
     <color rgba="0.3 0.3 0.3 1"/>
   </material>
+  <material name="yellow">
+    <color rgba="1 0.85 0 1"/>
+  </material>
 </robot>

File: grace_description/urdf/grace_gazebo.xacro (robot description, xacro)
@@ -159,3 +159,30 @@
     </sensor>
   </gazebo>
+  <!-- Camera Sensor -->
+  <gazebo reference="camera_link">
+    <sensor name="camera" type="camera">
+      <always_on>true</always_on>
+      <visualize>true</visualize>
+      <update_rate>30</update_rate>
+      <topic>camera/image_raw</topic>
+      <gz_frame_id>camera_optical_frame</gz_frame_id>
+      <camera>
+        <horizontal_fov>1.3962634</horizontal_fov>
+        <image>
+          <width>640</width>
+          <height>480</height>
+          <format>R8G8B8</format>
+        </image>
+        <clip>
+          <near>0.02</near>
+          <far>300</far>
+        </clip>
+        <noise>
+          <type>gaussian</type>
+          <mean>0.0</mean>
+          <stddev>0.007</stddev>
+        </noise>
+      </camera>
+    </sensor>
+  </gazebo>
 </robot>
